Commit message: Changes in launch and xacro files

File: r2p_foldy_base_description/urdf/r2p_foldy_base.xacro (robot description, xacro)
@@ -37,6 +37,6 @@
     </inertial>
   </link>
-  <!-- Camera Link -->
-  <link name="camera_link">
+  <!-- Realsense Camera Base Link -->
+  <link name="rs_cam_base_link">
     <visual>
       <origin xyz="0 0 0" rpy="${pi/2} 0 ${pi/2}"/>
@@ -60,8 +60,8 @@
     </inertial>
   </link>
-  <!-- Joint between Base Link and Camera Link -->
-  <joint name="base_camera_joint" type="fixed">
+  <!-- Joint between Base Link and Realsense Camera Base Link -->
+  <joint name="base_rs_cam_base_joint" type="fixed">
     <parent link="base_link"/>
-    <child link="camera_link"/>
+    <child link="rs_cam_base_link"/>
     <origin xyz="0.15 0 0.20" rpy="0 0 0"/>
     <axis xyz="1 0 0"/>

Commit message: New calculation of inverse kinematics

File: r2p_foldy_base_description/urdf/r2p_foldy_base.xacro (robot description, xacro)
@@ -38,5 +38,5 @@
   </link>
   <!-- Realsense Camera Base Link -->
-  <link name="rs_cam_base_link">
+  <link name="camera_link">
     <visual>
       <origin xyz="0 0 0" rpy="${pi/2} 0 ${pi/2}"/>
@@ -61,7 +61,7 @@
   </link>
   <!-- Joint between Base Link and Realsense Camera Base Link -->
-  <joint name="base_rs_cam_base_joint" type="fixed">
+  <joint name="base_camera_joint" type="fixed">
     <parent link="base_link"/>
-    <child link="rs_cam_base_link"/>
+    <child link="camera_link"/>
     <origin xyz="0.15 0 0.20" rpy="0 0 0"/>
     <axis xyz="1 0 0"/>

Commit message: New branch with minor changes

File: r2p_foldy_base_description/urdf/r2p_foldy_base.xacro (robot description, xacro)
@@ -14,4 +14,7 @@
     </inertial>
   </xacro:macro>
+  <!-- Dummy Link -->
+  <link name="dummy_link">
+  </link>
   <!-- Base Link -->
   <link name="base_link">
@@ -37,6 +40,13 @@
     </inertial>
   </link>
+  <!-- Joint between Dummy Link and Base Link -->
+  <joint name="dummy_base_joint" type="fixed">
+    <parent link="dummy_link"/>
+    <child link="base_link"/>
+    <origin xyz="0 0 -0.02" rpy="0 0 0"/>
+    <axis xyz="1 0 0"/>
+  </joint>
   <!-- Realsense Camera Base Link -->
-  <link name="camera_link">
+  <link name="rs_cam_base_link">
     <visual>
       <origin xyz="0 0 0" rpy="${pi/2} 0 ${pi/2}"/>
@@ -61,7 +71,7 @@
   </link>
   <!-- Joint between Base Link and Realsense Camera Base Link -->
-  <joint name="base_camera_joint" type="fixed">
+  <joint name="base_rs_cam_base_joint" type="fixed">
     <parent link="base_link"/>
-    <child link="camera_link"/>
+    <child link="rs_cam_base_link"/>
     <origin xyz="0.15 0 0.20" rpy="0 0 0"/>
     <axis xyz="1 0 0"/>
